File: Prototype V0.2/Prototype V0.2.brd (EAGLE design)
At the start: 35.7 x 22.5 mm, 15 parts

Commit message: adding the documentation here too
Parts:
- added IC1: 7805DT, linear4:TO252
- moved C3 6.52 mm to (16.6, 4.58)
- moved C2 5.02 mm to (24.4, 4.58)
- moved C4 3.50 mm to (32.2, 3.92)
- moved SV1 2.12 mm to (3.00, 5.50)
- moved D1 1.12 mm to (4.58, 15.0)
- moved R4 0.50 mm to (5.08, 19.6)
Connections:
- new net N$4: D1.A, IC1.2
- net GND: now also IC1.3
- net N$3: now also IC1.1; no longer D1.A
Routing:
- net GND: track 41.5 -> 33.1 mm
- net N$4: track 0.00 -> 7.57 mm
- net VIN: track 25.9 -> 18.9 mm
- net VCC: track 69.5 -> 63.8 mm
- net N$3: track 5.10 -> 9.84 mm
