File: Prototype V0.2/Prototype V0.2.sch (EAGLE design)
At the start: 15 parts

Commit message: adding the documentation here too
Parts:
- added IC1: 7805DT, linear4:7805DT
Connections:
- new net N$4: D1.A, IC1.VO
- net GND: now also IC1.GND
- net N$3: now also IC1.VI; no longer D1.A
Other:
- moved on the sheet: C2, C3, C4, D1, R1, R10, R4, R5, R6, R7, R8, R9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
